File: nfcid_reader/_autosave-nfcid_reader.kicad_pcb (KiCad board)
At the start: 2 copper layers, 91.4 x 43.2 mm, 20 parts, among them J1 BARREL_JACK, J2 ESP32_LEFT, J3 ESP32_RIGHT, J4 PN532, Q1 Q_PMOS_GSD, U1 MCP73832-2-OT, U2 LF33_TO220

Commit message: Minor fixes.
Parts:
- J2, J3: moved to F.Cu
- moved BT1 17.5 mm to (115.6, 110.5), turned to 180 degrees
- moved J1 1.27 mm to (108.0, 114.3), turned to 90 degrees
- moved Q1 1.27 mm to (97.8, 121.9)
- turned J2 to 180 degrees
- turned J3 to 180 degrees
Routing:
- net Net-(BT1-Pad1): track 32.4 -> 52.9 mm
- net GND: track 169.1 -> 156.2 mm
- net +5V: track 63.4 -> 69.8 mm
- net VCC: track 38.2 -> 39.5 mm
- removed copper zone on F.Cu, net GND
Other:
- board size 91.4 x 43.2 mm -> 83.8 x 43.2 mm
